Commit message: Added dummy values in the <inertial> tag

File: motoman_gp25_support/urdf/gp25_macro.xacro (robot description, xacro)
@@ -16,4 +16,8 @@
             </geometry>
         </collision>
+        <inertial>
+            <mass value="1"/>
+            <inertia ixx="1" ixy="0" ixz="0" iyy="1" iyz="0" izz="1"/>
+        </inertial>
     </link>
     <link name="${prefix}link_1_s">
@@ -29,4 +33,8 @@
             </geometry>
         </collision>
+        <inertial>
+            <mass value="1"/>
+            <inertia ixx="1" ixy="0" ixz="0" iyy="1" iyz="0" izz="1"/>
+        </inertial>
     </link>
     <link name="${prefix}link_2_l">
@@ -42,4 +50,8 @@
             </geometry>
         </collision>
+        <inertial>
+            <mass value="1"/>
+            <inertia ixx="1" ixy="0" ixz="0" iyy="1" iyz="0" izz="1"/>
+        </inertial>
     </link>
     <link name="${prefix}link_3_u">
@@ -55,4 +67,8 @@
             </geometry>
         </collision>
+        <inertial>
+            <mass value="1"/>
+            <inertia ixx="1" ixy="0" ixz="0" iyy="1" iyz="0" izz="1"/>
+        </inertial>
     </link>
     <link name="${prefix}link_4_r">
@@ -68,4 +84,8 @@
             </geometry>
         </collision>
+        <inertial>
+            <mass value="1"/>
+            <inertia ixx="1" ixy="0" ixz="0" iyy="1" iyz="0" izz="1"/>
+        </inertial>
     </link>
     <link name="${prefix}link_5_b">
@@ -81,4 +101,8 @@
             </geometry>
         </collision>
+        <inertial>
+            <mass value="1"/>
+            <inertia ixx="1" ixy="0" ixz="0" iyy="1" iyz="0" izz="1"/>
+        </inertial>
     </link>
     <link name="${prefix}link_6_t">
@@ -94,4 +118,8 @@
             </geometry>
         </collision>
+        <inertial>
+            <mass value="1"/>
+            <inertia ixx="1" ixy="0" ixz="0" iyy="1" iyz="0" izz="1"/>
+        </inertial>
     </link>
     <link name="${prefix}tool0"/>

Commit message: Gave more realistic, but still bogus, weights. The robot now doesn't fall over

File: motoman_gp25_support/urdf/gp25_macro.xacro (robot description, xacro)
@@ -17,5 +17,5 @@
         </collision>
         <inertial>
-            <mass value="1"/>
+            <mass value="100"/>
             <inertia ixx="1" ixy="0" ixz="0" iyy="1" iyz="0" izz="1"/>
         </inertial>
@@ -34,5 +34,5 @@
         </collision>
         <inertial>
-            <mass value="1"/>
+            <mass value="50"/>
             <inertia ixx="1" ixy="0" ixz="0" iyy="1" iyz="0" izz="1"/>
         </inertial>
@@ -51,5 +51,5 @@
         </collision>
         <inertial>
-            <mass value="1"/>
+            <mass value="25"/>
             <inertia ixx="1" ixy="0" ixz="0" iyy="1" iyz="0" izz="1"/>
         </inertial>
@@ -68,5 +68,5 @@
         </collision>
         <inertial>
-            <mass value="1"/>
+            <mass value="12"/>
             <inertia ixx="1" ixy="0" ixz="0" iyy="1" iyz="0" izz="1"/>
         </inertial>
@@ -85,5 +85,5 @@
         </collision>
         <inertial>
-            <mass value="1"/>
+            <mass value="6"/>
             <inertia ixx="1" ixy="0" ixz="0" iyy="1" iyz="0" izz="1"/>
         </inertial>
@@ -102,5 +102,5 @@
         </collision>
         <inertial>
-            <mass value="1"/>
+            <mass value="3"/>
             <inertia ixx="1" ixy="0" ixz="0" iyy="1" iyz="0" izz="1"/>
         </inertial>
