Commit message: Updated moveit config

File: motoman_gp25_moveit_config/config/motoman_gp25.ros2_control.xacro (robot description, xacro)
@@ -2,9 +2,8 @@
 <robot xmlns:xacro="http://www.ros.org/wiki/xacro">
     <xacro:macro name="motoman_gp25_ros2_control" params="name initial_positions_file">
-        <xacro:property name="initial_positions" value="${xacro.load_yaml(initial_positions_file)['initial_positions']}"/>
+        <xacro:property name="initial_positions" value="${load_yaml(initial_positions_file)['initial_positions']}"/>
         <ros2_control name="${name}" type="system">
             <hardware>
                 <!-- By default, set up controllers for simulation. This won't work on real hardware -->
-                <!--plugin>mock_components/GenericSystem</plugin-->
                 <plugin>ign_ros2_control/IgnitionSystem</plugin>
             </hardware>

File: motoman_gp25_moveit_config/config/motoman_gp25.urdf.xacro (robot description, xacro)
@@ -1,16 +1,16 @@
 <?xml version="1.0"?>
 <robot xmlns:xacro="http://www.ros.org/wiki/xacro" name="motoman_gp25">
-    <xacro:arg name="initial_positions_file" default="initial_positions.yaml" />
-    <!-- Import motoman_gp25 urdf file -->
-    <xacro:include filename="$(find motoman_gp25_support)/urdf/gp25.xacro" />
-    <!-- Import control_xacro -->
-    <xacro:include filename="motoman_gp25.ros2_control.xacro" />
-    <xacro:motoman_gp25_ros2_control name="FakeSystem" initial_positions_file="$(arg initial_positions_file)"/>
-    <gazebo reference="base_link"/>
-    <gazebo>
-      <plugin filename="libign_ros2_control-system.so" name="ign_ros2_control::IgnitionROS2ControlPlugin">
-        <parameters>$(find motoman_gp25_moveit_config)/config/ros2_controllers.yaml</parameters>
-        <controller_manager_node_name>controller_manager</controller_manager_node_name>
-      </plugin>
-    </gazebo>
+  <xacro:arg name="initial_positions_file" default="initial_positions.yaml" />
+  <!-- Import motoman_gp25 urdf file -->
+  <xacro:include filename="$(find motoman_gp25_support)/urdf/gp25.xacro" />
+  <!-- Import control_xacro -->
+  <xacro:include filename="motoman_gp25.ros2_control.xacro" />
+  <xacro:motoman_gp25_ros2_control name="FakeSystem" initial_positions_file="$(arg initial_positions_file)"/>
+  <gazebo reference="base_link"/>
+  <gazebo>
+    <plugin filename="libign_ros2_control-system.so" name="ign_ros2_control::IgnitionROS2ControlPlugin">
+      <parameters>$(find motoman_gp25_moveit_config)/config/ros2_controllers.yaml</parameters>
+      <controller_manager_node_name>controller_manager</controller_manager_node_name>
+    </plugin>
+  </gazebo>
 </robot>
